File: mk2/board_routed.kicad_pcb (KiCad board)
At the start: 2 copper layers, 258.1 x 122.5 mm, 85 parts, among them SW0 SW_Cherry_MX_1.00u_PCB, SW1 SW_Cherry_MX_1.00u_PCB, SW10 SW_Cherry_MX_1.00u_PCB, SW11 SW_Cherry_MX_1.00u_PCB, SW12 SW_Cherry_MX_1.00u_PCB, SW13 SW_Cherry_MX_1.00u_PCB, SW14 SW_Cherry_MX_1.00u_PCB, SW15 SW_Cherry_MX_1.00u_PCB, SW16 SW_Cherry_MX_1.00u_PCB, SW17 SW_Cherry_MX_1.00u_PCB, SW18 SW_Cherry_MX_1.00u_PCB, SW19 SW_Cherry_MX_1.00u_PCB, SW2 SW_Cherry_MX_1.00u_PCB, SW20 SW_Cherry_MX_1.00u_PCB, SW21 SW_Cherry_MX_1.00u_PCB, SW22 SW_Cherry_MX_1.00u_PCB, SW23 SW_Cherry_MX_1.00u_PCB, SW24 SW_Cherry_MX_1.00u_PCB, SW25 SW_Cherry_MX_1.00u_PCB, SW26 SW_Cherry_MX_1.00u_PCB, SW27 SW_Cherry_MX_1.00u_PCB, SW28 SW_Cherry_MX_1.00u_PCB, SW29 SW_Cherry_MX_1.00u_PCB, SW3 SW_Cherry_MX_1.00u_PCB, SW30 SW_Cherry_MX_1.00u_PCB, SW31 SW_Cherry_MX_1.00u_PCB, SW32 SW_Cherry_MX_1.00u_PCB, SW33 SW_Cherry_MX_1.00u_PCB, SW34 SW_Cherry_MX_1.00u_PCB, SW35 SW_Cherry_MX_1.00u_PCB, SW36 SW_Cherry_MX_1.00u_PCB, SW37 SW_Cherry_MX_1.00u_PCB, SW38 SW_Cherry_MX_1.00u_PCB, SW39 SW_Cherry_MX_1.00u_PCB, SW4 SW_Cherry_MX_1.00u_PCB, SW40 SW_Cherry_MX_1.00u_PCB, SW41 SW_Cherry_MX_1.00u_PCB, SW5 SW_Cherry_MX_1.00u_PCB, SW6 SW_Cherry_MX_1.00u_PCB, SW7 SW_Cherry_MX_1.00u_PCB, SW8 SW_Cherry_MX_1.00u_PCB, SW9 SW_Cherry_MX_1.00u_PCB

Commit message: Branding
Other:
- board text added: "flitter mk2 peterklein.dev"
- board text removed: "quine mk2 peterklein.dev"
Changed lines of the file:
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@@
   (gr_line (start 121.129977 138.364181) (end 121.0962 138.349524) (layer "Edge.Cuts") (width 0.1))
   (gr_line (start 273.988649 68.033411) (end 273.975822 68.067919) (layer "Edge.Cuts") (width 0.1))
-  (gr_text "quine mk2\npeterklein.dev" (at 226.809903 86.895798 39) (layer "F.SilkS")
+  (gr_text "flitter mk2\npeterklein.dev" (at 226.809903 86.895798 39) (layer "F.SilkS")
     (effects (font (size 1.27 1.27)))
   )

Commit message: Update kleinpa/keyboard-toolkit and add BOM generation
Parts:
- D0, D1, D10, D11, D12, D13, D14, D15, D16, D17, D18, D19, D2, D20, D21, D22, D23, D24, D25, D26, D27, D28, D29, D3, D30, D31, D32, D33, D34, D35, D36, D37, D38, D39, D4, D40, D41, D5, D6, D7, D8, D9: value D_SOD-123 -> 4148
